Commit message: Got soccerball to load at correct position, needed to change _sample_object in custom task

File: test/assets/soccerball.urdf (robot description, URDF)
Before this commit: robot urdf_robot, 1 links, 0 joints
Links:
- link baseLink: geometry collision mesh filename=soccerball.obj scale=.1 .1 .1; visual mesh filename=soccerball.obj scale=.1 .1 .1
